File: modified-sb-cnc-shield/sb-cnc-shield.kicad_pcb (KiCad board)
At the start: 2 copper layers, 68.6 x 53.3 mm, 63 parts, among them P1 XMOT, P2 YMOT, P3 ZMOT, P4 AMOT, P5 UART, P6 I2C, P7 ES_SETUP, P8 VMOT, SW1 RESET, U1 ARDUINO_UNO_SHIELD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

Commit message: add jack barrel for power supply in kicad
Parts:
- removed G***: LOGO, footprints:staticboards_logo
- JP19: value SE -> SpinEn
- JP20: value SD -> SpinDir
- JP21: value COOL -> CoolEn
- JP22: value ABORT -> Abort
- JP23: value HOLD -> Hold
- P8: value VMOT -> 12V-36V; footprint footprints:CONN_01x02_PITCH_5.08mm -> Connector_BarrelJack:BarrelJack_Horizontal
- moved P8 4.58 mm to (126.0, 111.2)
- moved U1 3.08 mm to (115.3, 117.0)
Connections:
- U1 pad 16: (no net) -> Net-(U1-Pad16)
- U1 pad 23: (no net) -> Net-(U1-Pad23)
Routing:
- net GNDA: track 166.5 -> 171.2 mm
- net VIN: track 126.7 -> 128.8 mm
