File: modified-sb-cnc-shield/sb-cnc-shield.sch (KiCad schematic (older format))
At the start: 62 parts, among them P1 XMOT, P2 YMOT, P3 ZMOT, P4 AMOT, P5 UART, P6 I2C, P7 ES_SETUP, P8 12V-36V, SW1 RESET, U1 ARDUINO_UNO_SHIELD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

Commit message: add jack barrel for power supply in kicad
Parts:
- removed P8: 12V-36V, footprints:CONN_01x02_PITCH_5.08mm, symbol sb-cnc-shield-rescue:CONN_01X02
- added P8: 12V-36V, symbol Connector_Generic:Conn_01x03
Connections:
- net GNDA: now also P8.2 (Pin_2), P8.3 (Pin_3)
- net VIN: now also P8.1 (Pin_1)
Changed lines of the file:
@@
 Connection ~ 3550 6100
-$Comp
-L sb-cnc-shield-rescue:CONN_01X02 P8
-U 1 1 564DCAAE
-P 2700 6950
-F 0 "P8" H 2700 7100 50  0000 C CNN
-F 1 "12V-36V" V 2800 6950 50  0000 C CNN
-F 2 "footprints:CONN_01x02_PITCH_5.08mm" H 2700 6950 60  0001 C CNN
-F 3 "" H 2700 6950 60  0000 C CNN
-	1    2700 6950
-	1    0    0    -1
-$EndComp
 $Comp
 L sb-cnc-shield-rescue:VIN #PWR038
@@
 Wire Wire Line
 	3550 6100 3550 6200
+$Comp
+L Connector_Generic:Conn_01x03 P8
+U 1 1 6176CCB3
+P 2700 7000
+F 0 "P8" H 2662 7199 50  0000 L CNN
+F 1 "12V-36V" V 2819 6833 50  0000 L CNN
+F 2 "" H 2700 7000 50  0001 C CNN
+F 3 "~" H 2700 7000 50  0001 C CNN
+	1    2700 7000
+	1    0    0    -1
+$EndComp
+Wire Wire Line
+	2500 7100 2500 7000
+Connection ~ 2500 7000
 $EndSCHEMATC
