File: mdified-sb-cnc-shield-master/sb-cnc-shield.sch (KiCad schematic (older format))
At the start: 62 parts, among them P1 XMOT, P2 YMOT, P3 ZMOT, P4 AMOT, P5 UART, P6 I2C, P7 ES_SETUP, P8 12V-36V, SW1 RESET, U1 ARDUINO_UNO_SHIELD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

Commit message: add jack barrel for power supply in kicad, correction
Parts:
- P8: footprint footprints:CONN_01x02_PITCH_5.08mm -> Connector_BarrelJack:BarrelJack_Horizontal; symbol sb-cnc-shield-rescue:CONN_01X02 -> Connector_Generic:Conn_01x03
Connections:
- net GNDA: now also P8.3 (Pin_3)
Changed lines of the file:
@@
 Connection ~ 3550 6100
 $Comp
-L sb-cnc-shield-rescue:CONN_01X02 P8
+L Connector_Generic:Conn_01x03 P8
 U 1 1 564DCAAE
-P 2700 6950
-F 0 "P8" H 2700 7100 50  0000 C CNN
-F 1 "12V-36V" V 2800 6950 50  0000 C CNN
-F 2 "footprints:CONN_01x02_PITCH_5.08mm" H 2700 6950 60  0001 C CNN
-F 3 "" H 2700 6950 60  0000 C CNN
-	1    2700 6950
+P 2700 7000
+F 0 "P8" H 2700 7229 50  0000 C CNN
+F 1 "12V-36V" V 2800 7000 50  0000 C CNN
+F 2 "Connector_BarrelJack:BarrelJack_Horizontal" H 2700 7000 60  0001 C CNN
+F 3 "" H 2700 7000 60  0000 C CNN
+	1    2700 7000
 	1    0    0    -1
 $EndComp
@@
 Wire Wire Line
 	3550 6100 3550 6200
+Wire Wire Line
+	2500 7100 2500 7000
+Connection ~ 2500 7000
 $EndSCHEMATC

Commit message: connect GNDs and connect the e-stop for reset
Parts:
- C1, C2, C3, C4: footprint Capacitors_SMD:c_elec_6.3x7.7 -> Capacitor_THT:C_Radial_D5.0mm_H11.0mm_P2.00mm
- P7: footprint Pin_Headers:Pin_Header_Straight_1x03 -> Connector_PinHeader_2.54mm:PinHeader_1x02_P2.54mm_Vertical; symbol sb-cnc-shield-rescue:CONN_01X03 -> Connector_Generic:Conn_01x02
Connections:
- net +5V: no longer P7.1 (P1)
- net GND: now also JP13.1, JP14.1, JP15.1, JP16.1, JP17.1, JP18.1, P7.1 (Pin_1); no longer P7.3 (P3)
- net RESET: now also P7.2 (Pin_2)
- removed net EN_SETUP: JP13.1, JP14.1, JP15.1, JP16.1, JP17.1, JP18.1, P7.2 (P2)
Changed lines of the file:
@@
 F 0 "C1" H 10875 2050 50  0000 L CNN
 F 1 "100uF" H 10900 1850 50  0000 L CNN
-F 2 "Capacitors_SMD:c_elec_6.3x7.7" H 10638 1800 30  0001 C CNN
+F 2 "Capacitor_THT:C_Radial_D5.0mm_H11.0mm_P2.00mm" H 10638 1800 30  0001 C CNN
 F 3 "" H 10850 1900 60  0000 C CNN
 	1    10850 1950
@@
 F 0 "C2" H 10875 3500 50  0000 L CNN
 F 1 "100uF" H 10900 3300 50  0000 L CNN
-F 2 "Capacitors_SMD:c_elec_6.3x7.7" H 10638 3250 30  0001 C CNN
+F 2 "Capacitor_THT:C_Radial_D5.0mm_H11.0mm_P2.00mm" H 10638 3250 30  0001 C CNN
 F 3 "" H 10850 3350 60  0000 C CNN
 	1    10850 3400
@@
 F 0 "C3" H 10875 4950 50  0000 L CNN
 F 1 "100uF" H 10900 4750 50  0000 L CNN
-F 2 "Capacitors_SMD:c_elec_6.3x7.7" H 10638 4700 30  0001 C CNN
+F 2 "Capacitor_THT:C_Radial_D5.0mm_H11.0mm_P2.00mm" H 10638 4700 30  0001 C CNN
 F 3 "" H 10850 4800 60  0000 C CNN
 	1    10850 4850
@@
 F 0 "C4" H 10875 6400 50  0000 L CNN
 F 1 "100uF" H 10900 6200 50  0000 L CNN
-F 2 "Capacitors_SMD:c_elec_6.3x7.7" H 10638 6150 30  0001 C CNN
+F 2 "Capacitor_THT:C_Radial_D5.0mm_H11.0mm_P2.00mm" H 10638 6150 30  0001 C CNN
 F 3 "" H 10850 6250 60  0000 C CNN
 	1    10850 6300
@@
 	5600 3750 5600 3650
 Connection ~ 5600 3650
-Text GLabel 5000 3250 0    39   Input ~ 0
-EN_SETUP
-Wire Wire Line
-	5000 3250 5100 3250
 Wire Wire Line
 	5100 3750 5250 3750
@@
 	5250 5250 5100 5250
 Connection ~ 5100 5250
-$Comp
-L sb-cnc-shield-rescue:CONN_01X03 P7
-U 1 1 564C03A6
-P 5850 6050
-F 0 "P7" H 5850 6250 50  0000 C CNN
-F 1 "ES_SETUP" V 5950 6050 50  0000 C CNN
-F 2 "Pin_Headers:Pin_Header_Straight_1x03" H 5850 6050 60  0001 C CNN
-F 3 "" H 5850 6050 60  0000 C CNN
-	1    5850 6050
-	1    0    0    -1
-$EndComp
-$Comp
-L power:GND #PWR030
-U 1 1 564C05A5
-P 5550 6250
-F 0 "#PWR030" H 5550 6000 50  0001 C CNN
-F 1 "GND" H 5550 6100 50  0000 C CNN
-F 2 "" H 5550 6250 60  0000 C CNN
-F 3 "" H 5550 6250 60  0000 C CNN
-	1    5550 6250
-	1    0    0    -1
-$EndComp
 $Comp
 L power:GND #PWR031
@@
 Wire Wire Line
 	8550 1050 8650 1050
-$Comp
-L power:+5V #PWR040
-U 1 1 564E12C2
-P 5550 5850
-F 0 "#PWR040" H 5550 5700 50  0001 C CNN
-F 1 "+5V" H 5550 5990 50  0000 C CNN
-F 2 "" H 5550 5850 60  0000 C CNN
-F 3 "" H 5550 5850 60  0000 C CNN
-	1    5550 5850
-	1    0    0    -1
-$EndComp
-Text GLabel 5450 6050 0    60   Input ~ 0
-EN_SETUP
-Wire Wire Line
-	5450 6050 5650 6050
-Wire Wire Line
-	5550 5950 5650 5950
-Wire Wire Line
-	5550 5850 5550 5950
-Wire Wire Line
-	5650 6150 5550 6150
-Wire Wire Line
-	5550 6150 5550 6250
+Text GLabel 5500 6150 0    60   Input ~ 0
+RESET
 Wire Wire Line
 	9250 6550 9450 6550
@@
 	2500 7100 2500 7000
 Connection ~ 2500 7000
+$Comp
+L Connector_Generic:Conn_01x02 P7
+U 1 1 564C03A6
+P 5850 6050
+F 0 "P7" H 5850 6250 50  0000 C CNN
+F 1 "ES_SETUP" V 5950 6050 50  0000 C CNN
+F 2 "Connector_PinHeader_2.54mm:PinHeader_1x02_P2.54mm_Vertical" H 5850 6050 60  0001 C CNN
+F 3 "" H 5850 6050 60  0000 C CNN
+	1    5850 6050
+	1    0    0    -1
+$EndComp
+$Comp
+L power:GND #PWR030
+U 1 1 564C05A5
+P 5650 6050
+F 0 "#PWR030" H 5650 5800 50  0001 C CNN
+F 1 "GND" V 5650 5900 50  0000 C CNN
+F 2 "" H 5650 6050 60  0000 C CNN
+F 3 "" H 5650 6050 60  0000 C CNN
+	1    5650 6050
+	0    1    -1   0
+$EndComp
+Wire Wire Line
+	5650 6150 5500 6150
+$Comp
+L power:GND #PWR?
+U 1 1 619427FF
+P 4700 3250
+F 0 "#PWR?" H 4700 3000 50  0001 C CNN
+F 1 "GND" V 4705 3122 50  0000 R CNN
+F 2 "" H 4700 3250 50  0001 C CNN
+F 3 "" H 4700 3250 50  0001 C CNN
+	1    4700 3250
+	0    1    1    0
+$EndComp
+Wire Wire Line
+	4700 3250 5100 3250
 $EndSCHEMATC
