File: PCBs/pick_n_place_head/pick_n_place_head/pick_n_place_head.kicad_pcb (KiCad board)
At the start: 2 copper layers, 63.2 x 43.1 mm, 10 parts, among them M1 magnet_conn_X5, M2 magnet_conn_X5, M3 magnet_conn_X5, U1 24AA02-OT

Commit message: modify kicad and freecad
Parts:
- moved R1 5.51 mm to (138.9, 64.7)
- moved blue1 5.24 mm to (145.4, 64.8), turned to 0 degrees
- moved R2 4.96 mm to (139.0, 69.8)
- moved green1 4.82 mm to (145.4, 69.7), turned to 0 degrees
Routing:
- net +3V3: track 53.0 -> 45.2 mm
- net GND: track 26.4 -> 31.0 mm
- net Net-(R1-Pad2): track 5.53 -> 8.11 mm
- net Net-(R2-Pad2): track 5.68 -> 8.06 mm
- net A2A: track 33.6 -> 34.7 mm
- net +12V: track 9.84 -> 8.86 mm
- added copper zone on F.Cu, net +3V3
- added copper zone on B.Cu, net GND
Other:
- net class +12V: clearance 0.2 -> 0.3; trace_width 0.7 -> 0.8; via_dia 0.8 -> 1
- net class Default: clearance 0.2 -> 0.3; trace_width 0.25 -> 0.4; via_dia 0.8 -> 1
- net class GND: clearance 0.2 -> 0.3; trace_width 0.7 -> 0.5; via_dia 0.8 -> 1
- rule trace_clearance: 0.2 -> 0.3
